Commit message: use mass as property instead and move sizes.xacro -> constants.xacro

File: description/constants.xacro (robot description, xacro)
@@ -5,7 +5,10 @@
   <xacro:property name="y_chassis_size" value="0.42" />
   <xacro:property name="z_chassis_size" value="0.14" />
+  <xacro:property name="chassis_mass" value="6" />
   <xacro:property name="drive_wheel_radius" value="0.102" />
   <xacro:property name="drive_wheel_length" value="0.04" />
+  <xacro:property name="drive_wheel_mass" value="3" />
   <xacro:property name="caster_wheel_radius" value="0.065" />
   <xacro:property name="caster_wheel_length" value="0.02" />
+  <xacro:property name="caster_wheel_mass" value="1" />
 </robot>

File: description/robot_core.xacro (robot description, xacro)
@@ -1,6 +1,8 @@
 <?xml version="1.0"?>
 <robot xmlns:xacro="http://www.ros.org/wiki/xacro">
+  <!-- INCLUDE -->
   <xacro:include filename="materials.xacro" />
-  <xacro:include filename="sizes.xacro" />
+  <xacro:include filename="constants.xacro" />
+  <xacro:include filename="inertial_macros.xacro" />
   <!-- BASE LINK-->
   <link name="base_link">
@@ -26,4 +28,8 @@
       </geometry>
     </collision>
+    <xacro:inertial_box mass="${chassis_mass}" x="${x_chassis_size}" y="${y_chassis_size}"
+      z="${z_chassis_size}">
+      <origin xyz="0 0 ${z_chassis_size/2}" />
+    </xacro:inertial_box>
   </link>
   <!-- LEFT WHEEL -->
@@ -46,4 +52,8 @@
       </geometry>
     </collision>
+    <xacro:inertial_cylinder mass="${drive_wheel_mass}" length="${drive_wheel_length}"
+      radius="${drive_wheel_radius}">
+      <origin xyz="0 0 0" rpy="0 0 0" />
+    </xacro:inertial_cylinder>
   </link>
   <!-- RIGHT WHEEL -->
@@ -66,4 +76,8 @@
       </geometry>
     </collision>
+    <xacro:inertial_cylinder mass="${drive_wheel_mass}" length="${drive_wheel_length}"
+      radius="${drive_wheel_radius}">
+      <origin xyz="0 0 0" rpy="0 0 0" />
+    </xacro:inertial_cylinder>
   </link>
   <!-- LEFT CASTER WHEELS -->
@@ -88,4 +102,8 @@
       </geometry>
     </collision>
+    <xacro:inertial_cylinder mass="${caster_wheel_mass}" length="${caster_wheel_length}"
+      radius="${caster_wheel_radius}">
+      <origin xyz="0 0 0" rpy="0 0 0" />
+    </xacro:inertial_cylinder>
   </link>
   <!-- RIGHT CASTER WHEELS -->
@@ -110,4 +128,8 @@
       </geometry>
     </collision>
+    <xacro:inertial_cylinder mass="${caster_wheel_mass}" length="${caster_wheel_length}"
+      radius="${caster_wheel_radius}">
+      <origin xyz="0 0 0" rpy="0 0 0" />
+    </xacro:inertial_cylinder>
   </link>
 </robot>
