Commit message: add gazebo urdf plugins

File: description/gazebo_control.xacro (robot description, xacro)
@@ -1,3 +1,25 @@
 <?xml version="1.0"?>
 <robot xmlns:xacro="http://www.ros.org/wiki/xacro">
+  <xacro:include filename="settings/frame_properties.xacro" />
+  <gazebo>
+    <plugin name="diff_drive" filename="libgazebo_ros_diff_drive.so">
+      <xacro:property name="wheel_separation"
+        value="${(y_chassis_size/2 + drive_wheel_length/2) * 2}" />
+      <!-- Wheel Informations-->
+      <left_joint>left_wheel_joint</left_joint>
+      <right_joint>right_wheel_joint</right_joint>
+      <wheel_separation>${(y_chassis_size/2 + drive_wheel_length/2) * 2}</wheel_separation>
+      <wheel_diameter>${drive_wheel_radius * 2}</wheel_diameter>
+      <!-- Limits -->
+      <!-- <max_wheel_torque>0.8825985</max_wheel_torque> -->
+      <max_wheel_torque>100</max_wheel_torque>
+      <max_accleration>5.0</max_accleration>
+      <!-- Outputs -->
+      <odometry_fram>odom</odometry_fram>
+      <robot_base_fram>base_link</robot_base_fram>
+      <publish_odom>true</publish_odom>
+      <publish_odom_tf>true</publish_odom_tf>
+      <publish_wheel_tf>true</publish_wheel_tf>
+    </plugin>
+  </gazebo>
 </robot>

Commit message: add max_wheel_torque and acceleration to frame_properties

File: description/gazebo_control.xacro (robot description, xacro)
@@ -13,6 +13,6 @@
       <!-- Limits -->
       <!-- <max_wheel_torque>0.8825985</max_wheel_torque> -->
-      <max_wheel_torque>100</max_wheel_torque>
-      <max_accleration>5.0</max_accleration>
+      <max_wheel_torque>${max_wheel_torque}</max_wheel_torque>
+      <max_accleration>${max_accleration}</max_accleration>
       <!-- Outputs -->
       <odometry_frame>odom</odometry_frame>

File: description/settings/frame_properties.xacro (robot description, xacro)
@@ -14,3 +14,6 @@
   <xacro:property name="caster_wheel_length" value="0.02" />
   <xacro:property name="caster_wheel_mass" value="1" />
+  <!-- SPEED -->
+  <xacro:property name="max_wheel_torque" value="100" />
+  <xacro:property name="max_acceleration" value="5.0" />
 </robot>
