Commit message: add chassis link and joint

File: description/robot.urdf.xacro (robot description, xacro)
@@ -1,6 +1,4 @@
 <?xml version="1.0"?>
 <robot xmlns:xacro="http://www.ros.org/wiki/xacro" name="robot">
-    <!-- Example link -->
-    <link name="base_link"></link>
     <xacro:include filename="robot_core.xacro" />
 </robot>

File: description/robot_core.xacro (robot description, xacro)
@@ -1,4 +1,5 @@
 <?xml version="1.0"?>
 <robot xmlns:xacro="http://www.ros.org/wiki/xacro">
+  <!-- material -->
   <material name="white">
     <color rgba="1 1 1 1" />
@@ -13,3 +14,21 @@
     <color rgba="0 0 0 1" />
   </material>
+  <!-- BASE LINK-->
+  <link name="base_link">
+  </link>
+  <!-- CHASSIS LINK -->
+  <joint name="chassis_joint" type="fixed">
+    <parent link="base_link" />
+    <child link="chassis" />
+    <origin xyz="-0.1 0 0 " />
+  </joint>
+  <link name="chassis">
+    <visual>
+      <origin xyz="0.25 0 0.07" />
+      <geometry>
+        <box size="0.5 0.42 0.14" />
+      </geometry>
+      <material name="white" />
+    </visual>
+  </link>
 </robot>

Commit message: add camera frame

File: description/robot.urdf.xacro (robot description, xacro)
@@ -15,3 +15,4 @@
     <xacro:include filename="robot_core.xacro" />
     <xacro:include filename="lidar.xacro" />
+    <xacro:include filename="camera.xacro" />
 </robot>

File: description/settings/frame_properties.xacro (robot description, xacro)
@@ -18,4 +18,9 @@
   <xacro:property name="lidar_frame_length" value="0.04" />
   <xacro:property name="lidar_mass" value="0.1" />
+  <!-- CAMERA -->
+  <xacro:property name="x_camera_size" value="0.05" />
+  <xacro:property name="y_camera_size" value="0.05" />
+  <xacro:property name="z_camera_size" value="0.05" />
+  <xacro:property name="camera_mass" value="0.1" />
   <!-- SPEED -->
   <xacro:property name="max_wheel_torque" value="100" />

Commit message: finish depth_camera xacro

File: description/robot.urdf.xacro (robot description, xacro)
@@ -15,4 +15,5 @@
     <xacro:include filename="robot_core.xacro" />
     <xacro:include filename="lidar.xacro" />
-    <xacro:include filename="camera.xacro" />
+    <!-- <xacro:include filename="camera.xacro" /> -->
+    <xacro:include filename="depth_camera.xacro" />
 </robot>

File: description/settings/frame_properties.xacro (robot description, xacro)
@@ -28,4 +28,7 @@
   <xacro:property name="min_view_range" value="0.05" />
   <xacro:property name="max_view_range" value="8.0" />
+  <!-- DEPTH-->
+  <xacro:property name="min_depth" value="0.1" />
+  <xacro:property name="max_depth" value="100.0" />
   <!-- SPEED -->
   <xacro:property name="max_wheel_torque" value="100" />

Commit message: unbreak gazebo

File: description/robot.urdf.xacro (robot description, xacro)
@@ -7,4 +7,5 @@
     <!-- PARAMS -->
     <xacro:arg name="use_ros2_control" default="true" />
+    <xacro:arg name="sim_mode" default="false" />
     <xacro:if value="$(arg use_ros2_control)">
         <xacro:include filename="ros2_control.xacro" />

File: description/ros2_control.xacro (robot description, xacro)
@@ -1,60 +1,62 @@
 <?xml version="1.0"?>
 <robot xmlns:xacro="http://www.ros.org/wiki/xacro">
-  <!-- <ros2_control name="GazeboSystem" type="system"> -->
-  <!--   <hardware> -->
-  <!--     <plugin>gazebo_ros2_control/GazeboSystem</plugin> -->
-  <!--   </hardware> -->
-  <!---->
-  <!--   <joint name="left_wheel_joint"> -->
-  <!--     <command_interface name="velocity"> -->
-  <!--       <param name="min">${wheel_min_speed}</param> -->
-  <!--       <param name="min">${wheel_max_speed}</param> -->
-  <!--     </command_interface> -->
-  <!--     <state_interface name="velocity" /> -->
-  <!--     <state_interface name="position" /> -->
-  <!--   </joint> -->
-  <!---->
-  <!--   <joint name="right_wheel_joint"> -->
-  <!--     <command_interface name="velocity"> -->
-  <!--       <param name="min">${wheel_min_speed}</param> -->
-  <!--       <param name="min">${wheel_max_speed}</param> -->
-  <!--     </command_interface> -->
-  <!--     <state_interface name="velocity" /> -->
-  <!--     <state_interface name="position" /> -->
-  <!--   </joint> -->
-  <!---->
-  <!-- </ros2_control> -->
-  <ros2_control name="RealRobot" type="system">
-    <hardware>
-      <plugin>diffdrive_arduino/DiffDriveArduino</plugin>
-      <param name="left_wheel_name">left_wheel_joint</param>
-      <param name="right_wheel_name">right_wheel_joint</param>
-      <param name="loop_rate">30</param>
-      <param name="device">/dev/ttyUSB0</param>
-      <param name="baud_rate">115200</param>
-      <param name="timeout">1000</param>
-      <param name="enc_counts_per_rev">3450</param>
-    </hardware>
-    <joint name="left_wheel_joint">
-      <command_interface name="velocity">
-        <param name="min">${wheel_min_speed}</param>
-        <param name="min">${wheel_max_speed}</param>
-      </command_interface>
-      <state_interface name="velocity" />
-      <state_interface name="position" />
-    </joint>
-    <joint name="right_wheel_joint">
-      <command_interface name="velocity">
-        <param name="min">${wheel_min_speed}</param>
-        <param name="min">${wheel_max_speed}</param>
-      </command_interface>
-      <state_interface name="velocity" />
-      <state_interface name="position" />
-    </joint>
-  </ros2_control>
+  <xacro:unless value="$(arg sim_mode)">
+    <ros2_control name="RealRobot" type="system">
+      <hardware>
+        <plugin>diffdrive_arduino/DiffDriveArduino</plugin>
+        <param name="left_wheel_name">left_wheel_joint</param>
+        <param name="right_wheel_name">right_wheel_joint</param>
+        <param name="loop_rate">30</param>
+        <param name="device">/dev/ttyUSB0</param>
+        <param name="baud_rate">115200</param>
+        <param name="timeout">1000</param>
+        <param name="enc_counts_per_rev">3450</param>
+      </hardware>
+      <joint name="left_wheel_joint">
+        <command_interface name="velocity">
+          <param name="min">${wheel_min_speed}</param>
+          <param name="min">${wheel_max_speed}</param>
+        </command_interface>
+        <state_interface name="velocity" />
+        <state_interface name="position" />
+      </joint>
+      <joint name="right_wheel_joint">
+        <command_interface name="velocity">
+          <param name="min">${wheel_min_speed}</param>
+          <param name="min">${wheel_max_speed}</param>
+        </command_interface>
+        <state_interface name="velocity" />
+        <state_interface name="position" />
+      </joint>
+    </ros2_control>
+  </xacro:unless>
+  <xacro:if value="$(arg sim_mode)">
+    <ros2_control name="GazeboSystem" type="system">
+      <hardware>
+        <plugin>gazebo_ros2_control/GazeboSystem</plugin>
+      </hardware>
+      <joint name="left_wheel_joint">
+        <command_interface name="velocity">
+          <param name="min">${wheel_min_speed}</param>
+          <param name="min">${wheel_max_speed}</param>
+        </command_interface>
+        <state_interface name="velocity" />
+        <state_interface name="position" />
+      </joint>
+      <joint name="right_wheel_joint">
+        <command_interface name="velocity">
+          <param name="min">${wheel_min_speed}</param>
+          <param name="min">${wheel_max_speed}</param>
+        </command_interface>
+        <state_interface name="velocity" />
+        <state_interface name="position" />
+      </joint>
+    </ros2_control>
+  </xacro:if>
   <!-- When not using Gazebo, we'll need to run `ros2 run controller_manager ros2_control_node` -->
   <gazebo>
     <plugin name="gazebo_ros2_control" filename="libgazebo_ros2_control.so">
       <parameters>$(find boom_bot)/config/my_controllers.yaml</parameters>
+      <parameters>$(find boom_bot)/config/gaz_ros2_ctl_use_sim.yaml</parameters>
     </plugin>
   </gazebo>
