Commit message: ros2_control add hardware interfaces

File: description/ros2_control.xacro (robot description, xacro)
@@ -8,7 +8,17 @@
     <joint name="left_wheel_joint">
       <command_interface name="velocity">
-        <param name="min">-10</param>
-        <param name="min">10</param>
+        <param name="min">${wheel_min_speed}</param>
+        <param name="min">${wheel_max_speed}</param>
       </command_interface>
+      <state_interface name="velocity" />
+      <state_interface name="position" />
+    </joint>
+    <joint name="right_wheel_joint">
+      <command_interface name="velocity">
+        <param name="min">${wheel_min_speed}</param>
+        <param name="min">${wheel_max_speed}</param>
+      </command_interface>
+      <state_interface name="velocity" />
+      <state_interface name="position" />
     </joint>
   </ros2_control>

File: description/settings/frame_properties.xacro (robot description, xacro)
@@ -17,3 +17,5 @@
   <xacro:property name="max_wheel_torque" value="100" />
   <xacro:property name="max_acceleration" value="5.0" />
+  <xacro:property name="wheel_max_speed" value="10.0" />
+  <xacro:property name="wheel_min_speed" value="-10.0" />
 </robot>

Commit message: add ros2_control xacro plugin

File: description/ros2_control.xacro (robot description, xacro)
@@ -1,7 +1,38 @@
 <?xml version="1.0"?>
 <robot xmlns:xacro="http://www.ros.org/wiki/xacro">
-  <ros2_control name="GazeboSystem" type="system">
+  <!-- <ros2_control name="GazeboSystem" type="system"> -->
+  <!--   <hardware> -->
+  <!--     <plugin>gazebo_ros2_control/GazeboSystem</plugin> -->
+  <!--   </hardware> -->
+  <!---->
+  <!--   <joint name="left_wheel_joint"> -->
+  <!--     <command_interface name="velocity"> -->
+  <!--       <param name="min">${wheel_min_speed}</param> -->
+  <!--       <param name="min">${wheel_max_speed}</param> -->
+  <!--     </command_interface> -->
+  <!--     <state_interface name="velocity" /> -->
+  <!--     <state_interface name="position" /> -->
+  <!--   </joint> -->
+  <!---->
+  <!--   <joint name="right_wheel_joint"> -->
+  <!--     <command_interface name="velocity"> -->
+  <!--       <param name="min">${wheel_min_speed}</param> -->
+  <!--       <param name="min">${wheel_max_speed}</param> -->
+  <!--     </command_interface> -->
+  <!--     <state_interface name="velocity" /> -->
+  <!--     <state_interface name="position" /> -->
+  <!--   </joint> -->
+  <!---->
+  <!-- </ros2_control> -->
+  <ros2_control name="RealRobot" type="system">
     <hardware>
-      <plugin>gazebo_ros2_control/GazeboSystem</plugin>
+      <plugin>diffdrive_arduino/DiffDriveArduino</plugin>
+      <param name="left_wheel_name">left_wheel_joint</param>
+      <param name="right_wheel_name">right_wheel_joint</param>
+      <param name="loop_rate">30</param>
+      <param name="device">/dev/ttyUSB0</param>
+      <param name="baud_rate">115200</param>
+      <param name="timeout">1000</param>
+      <param name="enc_counts_per_rev">3450</param>
     </hardware>
     <joint name="left_wheel_joint">

Commit message: use rotation spd for wheels min max spd and control plugin settings

File: description/ros2_control.xacro (robot description, xacro)
@@ -4,28 +4,24 @@
     <ros2_control name="RealRobot" type="system">
       <hardware>
-        <plugin>diffdrive_arduino/DiffDriveArduino</plugin>
+        <plugin>diffdrive_arduino/DiffDriveArduinoHardware</plugin>
         <param name="left_wheel_name">left_wheel_joint</param>
         <param name="right_wheel_name">right_wheel_joint</param>
-        <param name="loop_rate">30</param>
-        <param name="device">/dev/ttyUSB0</param>
+        <param name="device">/dev/serial/by-path/platform-fd500000.pcie-pci-0000:01:00.0-usb-0:1.3:1.0-port0</param>
         <param name="baud_rate">57600</param>
-        <param name="timeout">1000</param>
-        <param name="enc_counts_per_rev">3450</param>
+        <param name="timeout_ms">1000</param>
       </hardware>
-      <joint name="left_wheel_joint">
+      <joint name="${prefix}left_wheel_joint">
         <command_interface name="velocity">
           <param name="min">${wheel_min_speed}</param>
           <param name="min">${wheel_max_speed}</param>
         </command_interface>
-        <state_interface name="velocity" />
-        <state_interface name="position" />
+        <state_interface name="velocity"/>
       </joint>
-      <joint name="right_wheel_joint">
+      <joint name="${prefix}right_wheel_joint">
         <command_interface name="velocity">
           <param name="min">${wheel_min_speed}</param>
           <param name="min">${wheel_max_speed}</param>
         </command_interface>
-        <state_interface name="velocity" />
-        <state_interface name="position" />
+        <state_interface name="velocity"/>
       </joint>
     </ros2_control>

File: description/settings/frame_properties.xacro (robot description, xacro)
@@ -41,5 +41,6 @@
   <xacro:property name="max_wheel_torque" value="100" />
   <xacro:property name="max_acceleration" value="5.0" />
-  <xacro:property name="wheel_max_speed" value="275.0" />
-  <xacro:property name="wheel_min_speed" value="-275.0" />
+  <!-- ROTATION SPEED -->
+  <xacro:property name="wheel_max_speed" value="4.18" />
+  <xacro:property name="wheel_min_speed" value="-4.18" />
 </robot>

Commit message: fix description bug

File: description/ros2_control.xacro (robot description, xacro)
@@ -11,5 +11,5 @@
         <param name="timeout_ms">1000</param>
       </hardware>
-      <joint name="${prefix}left_wheel_joint">
+      <joint name="left_wheel_joint">
         <command_interface name="velocity">
           <param name="min">${wheel_min_speed}</param>
@@ -18,5 +18,5 @@
         <state_interface name="velocity"/>
       </joint>
-      <joint name="${prefix}right_wheel_joint">
+      <joint name="right_wheel_joint">
         <command_interface name="velocity">
           <param name="min">${wheel_min_speed}</param>
