Commit message: finish camear

File: description/camera.xacro (robot description, xacro)
@@ -1,12 +1,11 @@
 <?xml version="1.0"?>
 <robot xmlns:xacro="http://www.ros.org/wiki/xacro">
-  <!-- LASER -->
+  <!-- CAMERA -->
   <joint name="camera_joint" type="fixed">
     <parent link="chassis" />
     <child link="camera_link" />
-    <!-- <origin xyz="0 0 ${z_chassis_size}" rpy="0 0 0 " /> -->
-    <origin xyz="{(4*x_chassis_size) / 5} 0 ${z_chassis_size}" rpy="0 0 0 " />
+    <origin xyz="${(4*x_chassis_size) / 10} 0 ${z_chassis_size}" rpy="0 0 0 " />
   </joint>
-  <link name="laser_frame">
+  <link name="camera_link">
     <visual>
       <geometry>
@@ -25,31 +24,31 @@
     </xacro:inertial_box>
   </link>
+  <!-- CAMERA(OPTICAL)-->
+  <joint name="camera_optical_joint" type="fixed">
+    <parent link="camera_link" />
+    <child link="camera_link_optical" />
+    <origin xyz="0 0 0" rpy="${-pi/2} 0 ${-pi/2}" />
+  </joint>
+  <link name="camera_link_optical"></link>
   <gazebo reference="camera_link">
     <material>Gazebo/Red</material>
-    <sensor name="laser" type="ray">
+    <sensor name="camera" type="camera">
       <pose>0 0 0 0 0 0</pose>
       <visualize>true</visualize>
       <update_rate>10</update_rate>
-      <ray>
-        <scan>
-          <horizontal>
-            <samples>360</samples>
-            <resolution>1</resolution>
-            <min_angle>-3.14</min_angle>
-            <max_angle>3.14</max_angle>
-          </horizontal>
-        </scan>
-        <range>
-          <min>0.3</min>
-          <max>12.0</max>
-          <resolution>0.01</resolution>
-        </range>
-      </ray>
-      <plugin name="laser_controller" filename="libgazebo_ros_ray_sensor.so">
-        <ros>
-          <argument>~/out:=scan</argument>
-        </ros>
-        <output_type>sensor_msgs/LaserScan</output_type>
-        <frame_name>laser_frame</frame_name>
+      <camera>
+        <horizontal_fov>1.089</horizontal_fov>
+        <image>
+          <format>R8G8B8</format>
+          <width>1280</width>
+          <height>720</height>
+        </image>
+        <clip>
+          <near>0.05</near>
+          <far>8.0</far>
+        </clip>
+      </camera>
+      <plugin name="camera_controller" filename="libgazebo_ros_camera.so">
+        <frame_name>camera_link_optical</frame_name>
       </plugin>
     </sensor>

File: description/lidar.xacro (robot description, xacro)
@@ -5,5 +5,4 @@
     <parent link="chassis" />
     <child link="laser_frame" />
-    <!-- <origin xyz="0 0 ${z_chassis_size}" rpy="0 0 0 " /> -->
     <origin xyz="0 0 ${z_chassis_size}" rpy="0 0 0 " />
   </joint>

Commit message: move camera config to frame_properties.xacro

File: description/camera.xacro (robot description, xacro)
@@ -38,13 +38,13 @@
       <update_rate>10</update_rate>
       <camera>
-        <horizontal_fov>1.089</horizontal_fov>
+        <horizontal_fov>${horizontal_fov}</horizontal_fov>
         <image>
           <format>R8G8B8</format>
-          <width>1280</width>
-          <height>720</height>
+          <width>${frame_width}</width>
+          <height>${frame_height}</height>
         </image>
         <clip>
-          <near>0.05</near>
-          <far>8.0</far>
+          <near>${min_view_range}</near>
+          <far>${max_view_range}</far>
         </clip>
       </camera>

File: description/settings/frame_properties.xacro (robot description, xacro)
@@ -23,4 +23,9 @@
   <xacro:property name="z_camera_size" value="0.05" />
   <xacro:property name="camera_mass" value="0.1" />
+  <xacro:property name="horizontal_fov" value="1.089" />
+  <xacro:property name="frame_width" value="1280" />
+  <xacro:property name="frame_height" value="720" />
+  <xacro:property name="max_view_range" value="0.05" />
+  <xacro:property name="min_view_range" value="8.0" />
   <!-- SPEED -->
   <xacro:property name="max_wheel_torque" value="100" />

Commit message: change property name

File: description/camera.xacro (robot description, xacro)
@@ -41,6 +41,6 @@
         <image>
           <format>R8G8B8</format>
-          <width>${frame_width}</width>
-          <height>${frame_height}</height>
+          <width>${camera_frame_width}</width>
+          <height>${camera_frame_height}</height>
         </image>
         <clip>

File: description/settings/frame_properties.xacro (robot description, xacro)
@@ -24,6 +24,6 @@
   <xacro:property name="camera_mass" value="0.1" />
   <xacro:property name="horizontal_fov" value="1.089" />
-  <xacro:property name="frame_width" value="1280" />
-  <xacro:property name="frame_height" value="720" />
+  <xacro:property name="camera_frame_width" value="1280" />
+  <xacro:property name="camera_frame_height" value="720" />
   <xacro:property name="max_view_range" value="0.05" />
   <xacro:property name="min_view_range" value="8.0" />

Commit message: finish camaera

File: description/camera.xacro (robot description, xacro)
@@ -5,5 +5,5 @@
     <parent link="chassis" />
     <child link="camera_link" />
-    <origin xyz="${(4*x_chassis_size) / 10} 0 ${z_chassis_size}" rpy="0 0 0 " />
+    <origin xyz="${x_chassis_size/2} 0 ${z_chassis_size}" rpy="0 0 0 " />
   </joint>
   <link name="camera_link">

File: description/settings/frame_properties.xacro (robot description, xacro)
@@ -26,6 +26,6 @@
   <xacro:property name="camera_frame_width" value="1280" />
   <xacro:property name="camera_frame_height" value="720" />
-  <xacro:property name="max_view_range" value="0.05" />
-  <xacro:property name="min_view_range" value="8.0" />
+  <xacro:property name="min_view_range" value="0.05" />
+  <xacro:property name="max_view_range" value="8.0" />
   <!-- SPEED -->
   <xacro:property name="max_wheel_torque" value="100" />

Commit message: move cameras and lidar pos

File: description/camera.xacro (robot description, xacro)
@@ -5,5 +5,5 @@
     <parent link="chassis" />
     <child link="camera_link" />
-    <origin xyz="${x_chassis_size/2} 0 ${z_chassis_size}" rpy="0 0 0 " />
+    <origin xyz="${x_chassis_size/2} 0 ${z_chassis_size/2}" rpy="0 0 0 " />
   </joint>
   <link name="camera_link">

File: description/depth_camera.xacro (robot description, xacro)
@@ -5,5 +5,5 @@
     <parent link="chassis" />
     <child link="camera_link" />
-    <origin xyz="${x_chassis_size/2} 0 ${z_chassis_size}" rpy="0 0 0 " />
+    <origin xyz="${x_chassis_size/2} 0 ${z_chassis_size/2}" rpy="0 0 0 " />
   </joint>
   <link name="camera_link">

File: description/lidar.xacro (robot description, xacro)
@@ -5,5 +5,5 @@
     <parent link="chassis" />
     <child link="laser_frame" />
-    <origin xyz="0 0 ${z_chassis_size}" rpy="0 0 0 " />
+    <origin xyz="0 0 ${9*z_chassis_size/8}" rpy="0 0 0 " />
   </joint>
   <link name="laser_frame">

Commit message: update robot core

File: description/camera.xacro (robot description, xacro)
@@ -3,7 +3,7 @@
   <!-- CAMERA -->
   <joint name="camera_joint" type="fixed">
-    <parent link="chassis" />
+    <parent link="handle" />
     <child link="camera_link" />
-    <origin xyz="${x_chassis_size/2} 0 ${z_chassis_size/2}" rpy="0 0 0 " />
+    <origin xyz="${x_handle_size/2} 0 ${17*z_handle_size/20}" rpy="0 0 0 " />
   </joint>
   <link name="camera_link">

File: description/depth_camera.xacro (robot description, xacro)
@@ -3,7 +3,7 @@
   <!-- CAMERA -->
   <joint name="camera_joint" type="fixed">
-    <parent link="chassis" />
+    <parent link="handle" />
     <child link="camera_link" />
-    <origin xyz="${x_chassis_size/2} 0 ${z_chassis_size/2}" rpy="0 0 0 " />
+    <origin xyz="${x_handle_size/2} 0 ${17*z_handle_size/20}" rpy="0 0 0 " />
   </joint>
   <link name="camera_link">

File: description/lidar.xacro (robot description, xacro)
@@ -3,7 +3,7 @@
   <!-- LASER -->
   <joint name="laser_joint" type="fixed">
-    <parent link="chassis" />
+    <parent link="handle" />
     <child link="laser_frame" />
-    <origin xyz="0 0 ${9*z_chassis_size/8}" rpy="0 0 0 " />
+    <origin xyz="0 0 ${z_handle_size + 0.02}" rpy="0 0 0 " />
   </joint>
   <link name="laser_frame">

File: description/robot_core.xacro (robot description, xacro)
@@ -41,5 +41,5 @@
     <parent link="chassis" />
     <child link="handle" />
-    <origin xyz="-${x_chassis_size/2 + x_handle_size/2} 0 0" />
+    <origin xyz="${-x_chassis_size/2} 0 0" />
   </joint>
   <link name="handle">
@@ -66,5 +66,6 @@
     <parent link="base_link" />
     <child link="left_wheel" />
-    <origin xyz="0 ${y_chassis_size/2 + drive_wheel_length/2} 0" rpy="-${pi/2} 0 0" />
+    <origin xyz="-${2*x_chassis_size /6} ${y_chassis_size/2 + drive_wheel_length/2} 0"
+      rpy="-${pi/2} 0 0" />
     <axis xyz="0 0 1" />
   </joint>
@@ -93,5 +94,6 @@
     <parent link="base_link" />
     <child link="right_wheel" />
-    <origin xyz="0 -${y_chassis_size/2 + drive_wheel_length/2} 0" rpy="${pi/2} 0 0" />
+    <origin xyz="-${2*x_chassis_size /6} -${y_chassis_size/2 + drive_wheel_length/2} 0"
+      rpy="${pi/2} 0 0" />
     <axis xyz="0 0 -1" />
   </joint>
