Commit message: use chassis size as a property instead

File: description/robot_core.xacro (robot description, xacro)
@@ -14,4 +14,8 @@
     <color rgba="0 0 0 1" />
   </material>
+  <!-- SIZE -->
+  <xacro:property name="x_chassis_size" value="0.5" />
+  <xacro:property name="y_chassis_size" value="0.42" />
+  <xacro:property name="z_chassis_size" value="0.14" />
   <!-- BASE LINK-->
   <link name="base_link">
@@ -25,7 +29,7 @@
   <link name="chassis">
     <visual>
-      <origin xyz="0.25 0 0.07" />
+      <origin xyz="${x_chassis_size/2} 0 ${z_chassis_size/2}" />
       <geometry>
-        <box size="0.5 0.42 0.14" />
+        <box size="${x_chassis_size} ${y_chassis_size} ${z_chassis_size}" />
       </geometry>
       <material name="white" />

Commit message: add left and right wheels

File: description/robot_core.xacro (robot description, xacro)
@@ -18,4 +18,6 @@
   <xacro:property name="y_chassis_size" value="0.42" />
   <xacro:property name="z_chassis_size" value="0.14" />
+  <xacro:property name="drive_wheel_radius" value="0.102" />
+  <xacro:property name="drive_wheel_length" value="0.04" />
   <!-- BASE LINK-->
   <link name="base_link">
@@ -36,3 +38,33 @@
     </visual>
   </link>
+  <!-- LEFT WHEEL -->
+  <joint name="left_wheel_joint" type="continuous">
+    <parent link="base_link" />
+    <child link="left_wheel" />
+    <origin xyz="0 ${y_chassis_size/2 + drive_wheel_length/2} 0" rpy="-${pi/2} 0 0" />
+    <axis xyz="0 0 1" />
+  </joint>
+  <link name="left_wheel">
+    <visual>
+      <geometry>
+        <cylinder radius="${drive_wheel_radius}" length="${drive_wheel_length}" />
+      </geometry>
+      <material name="blue" />
+    </visual>
+  </link>
+  <!-- RIGHT WHEEL -->
+  <joint name="right_wheel_joint" type="continuous">
+    <parent link="base_link" />
+    <child link="right_wheel" />
+    <origin xyz="0 -${y_chassis_size/2 + drive_wheel_length/2} 0" rpy="${pi/2} 0 0" />
+    <axis xyz="0 0 -1" />
+  </joint>
+  <link name="right_wheel">
+    <visual>
+      <geometry>
+        <cylinder radius="${drive_wheel_radius}" length="${drive_wheel_length}" />
+      </geometry>
+      <material name="blue" />
+    </visual>
+  </link>
 </robot>

Commit message: centered the drive wheels

File: description/robot_core.xacro (robot description, xacro)
@@ -27,9 +27,9 @@
     <parent link="base_link" />
     <child link="chassis" />
-    <origin xyz="-0.1 0 0 " />
+    <origin xyz="0 0 0 " />
   </joint>
   <link name="chassis">
     <visual>
-      <origin xyz="${x_chassis_size/2} 0 ${z_chassis_size/2}" />
+      <origin xyz="0 0 ${z_chassis_size/2}" />
       <geometry>
         <box size="${x_chassis_size} ${y_chassis_size} ${z_chassis_size}" />

Commit message: add caster wheels

File: description/robot_core.xacro (robot description, xacro)
@@ -20,4 +20,6 @@
   <xacro:property name="drive_wheel_radius" value="0.102" />
   <xacro:property name="drive_wheel_length" value="0.04" />
+  <xacro:property name="caster_wheel_radius" value="0.065" />
+  <xacro:property name="caster_wheel_length" value="0.02" />
   <!-- BASE LINK-->
   <link name="base_link">
@@ -68,3 +70,37 @@
     </visual>
   </link>
+  <!-- LEFT CASTER WHEELS -->
+  <joint name="left_caster_wheel_joint" type="fixed">
+    <parent link="base_link" />
+    <child link="left_caster_wheel" />
+    <origin
+      xyz="${2*x_chassis_size /6} ${2*y_chassis_size/5} -${drive_wheel_radius - caster_wheel_radius}"
+      rpy="-${pi/2} 0 0" />
+    <axis xyz="0 0 1" />
+  </joint>
+  <link name="left_caster_wheel">
+    <visual>
+      <geometry>
+        <cylinder radius="${caster_wheel_radius}" length="${caster_wheel_length}" />
+      </geometry>
+      <material name="black" />
+    </visual>
+  </link>
+  <!-- RIGHT CASTER WHEELS -->
+  <joint name="right_caster_wheel_joint" type="fixed">
+    <parent link="base_link" />
+    <child link="right_caster_wheel" />
+    <origin
+      xyz="${2*x_chassis_size /6} -${2*y_chassis_size/5} -${drive_wheel_radius - caster_wheel_radius}"
+      rpy="${pi/2} 0 0" />
+    <axis xyz="0 0 -1" />
+  </joint>
+  <link name="right_caster_wheel">
+    <visual>
+      <geometry>
+        <cylinder radius="${caster_wheel_radius}" length="${caster_wheel_length}" />
+      </geometry>
+      <material name="black" />
+    </visual>
+  </link>
 </robot>

Commit message: add collisions

File: description/robot_core.xacro (robot description, xacro)
@@ -39,4 +39,10 @@
       <material name="white" />
     </visual>
+    <collision>
+      <origin xyz="0 0 ${z_chassis_size/2}" />
+      <geometry>
+        <box size="${x_chassis_size} ${y_chassis_size} ${z_chassis_size}" />
+      </geometry>
+    </collision>
   </link>
   <!-- LEFT WHEEL -->
@@ -54,4 +60,9 @@
       <material name="blue" />
     </visual>
+    <collision>
+      <geometry>
+        <cylinder radius="${drive_wheel_radius}" length="${drive_wheel_length}" />
+      </geometry>
+    </collision>
   </link>
   <!-- RIGHT WHEEL -->
@@ -69,4 +80,9 @@
       <material name="blue" />
     </visual>
+    <collision>
+      <geometry>
+        <cylinder radius="${drive_wheel_radius}" length="${drive_wheel_length}" />
+      </geometry>
+    </collision>
   </link>
   <!-- LEFT CASTER WHEELS -->
@@ -86,4 +102,9 @@
       <material name="black" />
     </visual>
+    <collision>
+      <geometry>
+        <cylinder radius="${caster_wheel_radius}" length="${caster_wheel_length}" />
+      </geometry>
+    </collision>
   </link>
   <!-- RIGHT CASTER WHEELS -->
@@ -103,4 +124,9 @@
       <material name="black" />
     </visual>
+    <collision>
+      <geometry>
+        <cylinder radius="${caster_wheel_radius}" length="${caster_wheel_length}" />
+      </geometry>
+    </collision>
   </link>
 </robot>

Commit message: move defined materials to materials.xacro

File: description/robot_core.xacro (robot description, xacro)
@@ -1,25 +1,5 @@
 <?xml version="1.0"?>
 <robot xmlns:xacro="http://www.ros.org/wiki/xacro">
-  <!-- material -->
-  <material name="white">
-    <color rgba="1 1 1 1" />
-  </material>
-  <material name="orange">
-    <color rgba="1 0.3 0.1 1" />
-  </material>
-  <material name="blue">
-    <color rgba="0.2 0.2 1 1" />
-  </material>
-  <material name="black">
-    <color rgba="0 0 0 1" />
-  </material>
-  <!-- SIZE -->
-  <xacro:property name="x_chassis_size" value="0.5" />
-  <xacro:property name="y_chassis_size" value="0.42" />
-  <xacro:property name="z_chassis_size" value="0.14" />
-  <xacro:property name="drive_wheel_radius" value="0.102" />
-  <xacro:property name="drive_wheel_length" value="0.04" />
-  <xacro:property name="caster_wheel_radius" value="0.065" />
-  <xacro:property name="caster_wheel_length" value="0.02" />
+  <xacro:include filename="materials.xacro" />
   <!-- BASE LINK-->
   <link name="base_link">

Commit message: add gazebo ref in robot_core

File: description/robot_core.xacro (robot description, xacro)
@@ -33,4 +33,7 @@
     </xacro:inertial_box>
   </link>
+  <gazebo reference="chassis">
+    <material name="white" />
+  </gazebo>
   <!-- LEFT WHEEL -->
   <joint name="left_wheel_joint" type="continuous">
@@ -57,4 +60,7 @@
     </xacro:inertial_cylinder>
   </link>
+  <gazebo reference="left_wheel">
+    <material name="blue" />
+  </gazebo>
   <!-- RIGHT WHEEL -->
   <joint name="right_wheel_joint" type="continuous">
@@ -81,4 +87,7 @@
     </xacro:inertial_cylinder>
   </link>
+  <gazebo reference="right_wheel">
+    <material name="blue" />
+  </gazebo>
   <!-- LEFT CASTER WHEELS -->
   <joint name="left_caster_wheel_joint" type="fixed">
@@ -106,4 +115,7 @@
       <origin xyz="0 0 0" rpy="0 0 0" />
     </xacro:inertial_cylinder>
+    <gazebo reference="left_caster_wheel">
+      <material name="black" />
+    </gazebo>
   </link>
   <!-- RIGHT CASTER WHEELS -->
@@ -132,4 +144,7 @@
       <origin xyz="0 0 0" rpy="0 0 0" />
     </xacro:inertial_cylinder>
+    <gazebo reference="right_caster_wheel">
+      <material name="black" />
+    </gazebo>
   </link>
 </robot>

Commit message: fix color bug

File: description/robot_core.xacro (robot description, xacro)
@@ -34,5 +34,5 @@
   </link>
   <gazebo reference="chassis">
-    <material name="white" />
+    <material>Gazebo/White</material>
   </gazebo>
   <!-- LEFT WHEEL -->
@@ -61,5 +61,5 @@
   </link>
   <gazebo reference="left_wheel">
-    <material name="blue" />
+    <material>Gazebo/Blue</material>
   </gazebo>
   <!-- RIGHT WHEEL -->
@@ -88,5 +88,5 @@
   </link>
   <gazebo reference="right_wheel">
-    <material name="blue" />
+    <material>Gazebo/Blue</material>
   </gazebo>
   <!-- LEFT CASTER WHEELS -->
@@ -115,8 +115,8 @@
       <origin xyz="0 0 0" rpy="0 0 0" />
     </xacro:inertial_cylinder>
-    <gazebo reference="left_caster_wheel">
-      <material name="black" />
-    </gazebo>
   </link>
+  <gazebo reference="left_caster_wheel">
+    <material>Gazebo/Black</material>
+  </gazebo>
   <!-- RIGHT CASTER WHEELS -->
   <joint name="right_caster_wheel_joint" type="fixed">
@@ -144,7 +144,7 @@
       <origin xyz="0 0 0" rpy="0 0 0" />
     </xacro:inertial_cylinder>
-    <gazebo reference="right_caster_wheel">
-      <material name="black" />
-    </gazebo>
   </link>
+  <gazebo reference="right_caster_wheel">
+    <material>Gazebo/Black</material>
+  </gazebo>
 </robot>

Commit message: add 2 back_wheels

File: description/robot_core.xacro (robot description, xacro)
@@ -90,8 +90,8 @@
     <material>Gazebo/Blue</material>
   </gazebo>
-  <!-- LEFT CASTER WHEELS -->
-  <joint name="left_caster_wheel_joint" type="fixed">
-    <parent link="base_link" />
-    <child link="left_caster_wheel" />
+  <!-- FRONT LEFT CASTER WHEELS -->
+  <joint name="front_left_caster_wheel_joint" type="fixed">
+    <parent link="base_link" />
+    <child link="front_left_caster_wheel" />
     <origin
       xyz="${2*x_chassis_size /6} ${2*y_chassis_size/5} -${drive_wheel_radius - caster_wheel_radius}"
@@ -99,30 +99,30 @@
     <axis xyz="0 0 1" />
   </joint>
-  <link name="left_caster_wheel">
-    <visual>
-      <geometry>
-        <cylinder radius="${caster_wheel_radius}" length="${caster_wheel_length}" />
-      </geometry>
-      <material name="black" />
-    </visual>
-    <collision>
-      <geometry>
-        <cylinder radius="${caster_wheel_radius}" length="${caster_wheel_length}" />
-      </geometry>
-    </collision>
-    <xacro:inertial_cylinder mass="${caster_wheel_mass}" length="${caster_wheel_length}"
-      radius="${caster_wheel_radius}">
-      <origin xyz="0 0 0" rpy="0 0 0" />
-    </xacro:inertial_cylinder>
-  </link>
-  <gazebo reference="left_caster_wheel">
-    <material>Gazebo/Black</material>
-    <mu1 value="0.001" />
-    <mu2 value="0.001" />
-  </gazebo>
-  <!-- RIGHT CASTER WHEELS -->
-  <joint name="right_caster_wheel_joint" type="fixed">
-    <parent link="base_link" />
-    <child link="right_caster_wheel" />
+  <link name="front_left_caster_wheel">
+    <visual>
+      <geometry>
+        <cylinder radius="${caster_wheel_radius}" length="${caster_wheel_length}" />
+      </geometry>
+      <material name="black" />
+    </visual>
+    <collision>
+      <geometry>
+        <cylinder radius="${caster_wheel_radius}" length="${caster_wheel_length}" />
+      </geometry>
+    </collision>
+    <xacro:inertial_cylinder mass="${caster_wheel_mass}" length="${caster_wheel_length}"
+      radius="${caster_wheel_radius}">
+      <origin xyz="0 0 0" rpy="0 0 0" />
+    </xacro:inertial_cylinder>
+  </link>
+  <gazebo reference="front_left_caster_wheel">
+    <material>Gazebo/Black</material>
+    <mu1 value="0.001" />
+    <mu2 value="0.001" />
+  </gazebo>
+  <!-- FRONT RIGHT CASTER WHEELS -->
+  <joint name="front_right_caster_wheel_joint" type="fixed">
+    <parent link="base_link" />
+    <child link="front_right_caster_wheel" />
     <origin
       xyz="${2*x_chassis_size /6} -${2*y_chassis_size/5} -${drive_wheel_radius - caster_wheel_radius}"
@@ -130,22 +130,84 @@
     <axis xyz="0 0 -1" />
   </joint>
-  <link name="right_caster_wheel">
-    <visual>
-      <geometry>
-        <cylinder radius="${caster_wheel_radius}" length="${caster_wheel_length}" />
-      </geometry>
-      <material name="black" />
-    </visual>
-    <collision>
-      <geometry>
-        <cylinder radius="${caster_wheel_radius}" length="${caster_wheel_length}" />
-      </geometry>
-    </collision>
-    <xacro:inertial_cylinder mass="${caster_wheel_mass}" length="${caster_wheel_length}"
-      radius="${caster_wheel_radius}">
-      <origin xyz="0 0 0" rpy="0 0 0" />
-    </xacro:inertial_cylinder>
-  </link>
-  <gazebo reference="right_caster_wheel">
+  <link name="front_right_caster_wheel">
+    <visual>
+      <geometry>
+        <cylinder radius="${caster_wheel_radius}" length="${caster_wheel_length}" />
+      </geometry>
+      <material name="black" />
+    </visual>
+    <collision>
+      <geometry>
+        <cylinder radius="${caster_wheel_radius}" length="${caster_wheel_length}" />
+      </geometry>
+    </collision>
+    <xacro:inertial_cylinder mass="${caster_wheel_mass}" length="${caster_wheel_length}"
+      radius="${caster_wheel_radius}">
+      <origin xyz="0 0 0" rpy="0 0 0" />
+    </xacro:inertial_cylinder>
+  </link>
+  <gazebo reference="front_right_caster_wheel">
+    <material>Gazebo/Black</material>
+    <mu1 value="0.001" />
+    <mu2 value="0.001" />
+  </gazebo>
+  <!-- BACK LEFT CASTER WHEELS -->
+  <joint name="back_left_caster_wheel_joint" type="fixed">
+    <parent link="base_link" />
+    <child link="back_left_caster_wheel" />
+    <origin
+      xyz="-${2*x_chassis_size /6} ${2*y_chassis_size/5} -${drive_wheel_radius - caster_wheel_radius}"
+      rpy="-${pi/2} 0 0" />
+    <axis xyz="0 0 1" />
+  </joint>
+  <link name="back_left_caster_wheel">
+    <visual>
+      <geometry>
+        <cylinder radius="${caster_wheel_radius}" length="${caster_wheel_length}" />
+      </geometry>
+      <material name="black" />
+    </visual>
+    <collision>
+      <geometry>
+        <cylinder radius="${caster_wheel_radius}" length="${caster_wheel_length}" />
+      </geometry>
+    </collision>
+    <xacro:inertial_cylinder mass="${caster_wheel_mass}" length="${caster_wheel_length}"
+      radius="${caster_wheel_radius}">
+      <origin xyz="0 0 0" rpy="0 0 0" />
+    </xacro:inertial_cylinder>
+  </link>
+  <gazebo reference="back_left_caster_wheel">
+    <material>Gazebo/Black</material>
+    <mu1 value="0.001" />
+    <mu2 value="0.001" />
+  </gazebo>
+  <!-- BACK RIGHT CASTER WHEELS -->
+  <joint name="back_right_caster_wheel_joint" type="fixed">
+    <parent link="base_link" />
+    <child link="back_right_caster_wheel" />
+    <origin
+      xyz="-${2*x_chassis_size /6} -${2*y_chassis_size/5} -${drive_wheel_radius - caster_wheel_radius}"
+      rpy="${pi/2} 0 0" />
+    <axis xyz="0 0 -1" />
+  </joint>
+  <link name="back_right_caster_wheel">
+    <visual>
+      <geometry>
+        <cylinder radius="${caster_wheel_radius}" length="${caster_wheel_length}" />
+      </geometry>
+      <material name="black" />
+    </visual>
+    <collision>
+      <geometry>
+        <cylinder radius="${caster_wheel_radius}" length="${caster_wheel_length}" />
+      </geometry>
+    </collision>
+    <xacro:inertial_cylinder mass="${caster_wheel_mass}" length="${caster_wheel_length}"
+      radius="${caster_wheel_radius}">
+      <origin xyz="0 0 0" rpy="0 0 0" />
+    </xacro:inertial_cylinder>
+  </link>
+  <gazebo reference="back_right_caster_wheel">
     <material>Gazebo/Black</material>
     <mu1 value="0.001" />

Commit message: add robot's base_footprint link

File: description/robot_core.xacro (robot description, xacro)
@@ -4,4 +4,12 @@
   <link name="base_link">
   </link>
+  <!-- BASE_FOOTPRINT LINK-->
+  <joint name="base_footprint_joint" type="fixed">
+    <parent link="base_link" />
+    <child link="base_footprint" />
+    <origin xyz="0 0 0" />
+  </joint>
+  <link name="base_footprint">
+  </link>
   <!-- CHASSIS LINK -->
   <joint name="chassis_joint" type="fixed">

Commit message: update size and add handle

File: description/robot_core.xacro (robot description, xacro)
@@ -37,7 +37,29 @@
     </xacro:inertial_box>
   </link>
-  <gazebo reference="chassis">
-    <material>Gazebo/White</material>
-  </gazebo>
+  <!-- HANDLE -->
+  <joint name="handle_joint" type="fixed">
+    <parent link="chassis" />
+    <child link="handle" />
+    <origin xyz="-${x_chassis_size/2 + x_handle_size/2} 0 0" />
+  </joint>
+  <link name="handle">
+    <visual>
+      <origin xyz="0 0 ${z_handle_size/2}" />
+      <geometry>
+        <box size="${x_handle_size} ${y_handle_size} ${z_handle_size}" />
+      </geometry>
+      <material name="white" />
+    </visual>
+    <collision>
+      <origin xyz="0 0 ${z_handle_size/2}" />
+      <geometry>
+        <box size="${x_handle_size} ${y_handle_size} ${z_handle_size}" />
+      </geometry>
+    </collision>
+    <xacro:inertial_box mass="${handle_mass}" x="${x_handle_size}" y="${y_handle_size}"
+      z="${z_handle_size}">
+      <origin xyz="0 0 0" />
+    </xacro:inertial_box>
+  </link>
   <!-- LEFT WHEEL -->
   <joint name="left_wheel_joint" type="continuous">

File: description/settings/frame_properties.xacro (robot description, xacro)
@@ -5,11 +5,15 @@
   <xacro:property name="y_chassis_size" value="0.42" />
   <xacro:property name="z_chassis_size" value="0.14" />
-  <xacro:property name="chassis_mass" value="6" />
+  <xacro:property name="chassis_mass" value="4.4" />
+  <xacro:property name="x_handle_size" value="0.13" />
+  <xacro:property name="y_handle_size" value="0.42" />
+  <xacro:property name="z_handle_size" value="0.8" />
+  <xacro:property name="handle_mass" value="3" />
   <!-- DRIVE WHEELS-->
   <xacro:property name="drive_wheel_radius" value="0.102" />
   <xacro:property name="drive_wheel_length" value="0.04" />
-  <xacro:property name="drive_wheel_mass" value="3" />
+  <xacro:property name="drive_wheel_mass" value="2" />
   <!-- CASTER WHEELS-->
-  <xacro:property name="caster_wheel_radius" value="0.065" />
+  <xacro:property name="caster_wheel_radius" value="0.055" />
   <xacro:property name="caster_wheel_length" value="0.02" />
   <xacro:property name="caster_wheel_mass" value="1" />

Commit message: finish frame update

File: description/robot_core.xacro (robot description, xacro)
@@ -62,9 +62,35 @@
     </xacro:inertial_box>
   </link>
+  <!-- LEFT MOTOR -->
+  <joint name="left_motor_joint" type="continuous">
+    <parent link="base_link" />
+    <child link="left_motor" />
+    <origin xyz="-${2*x_chassis_size /6} -${y_chassis_size/2} 0"
+      rpy="0 0 0" />
+    <axis xyz="0 0 -1" />
+  </joint>
+  <link name="left_motor">
+    <visual>
+      <geometry>
+        <box size="${x_motor_size} ${y_motor_size} ${z_motor_size}" />
+      </geometry>
+      <material name="blue" />
+    </visual>
+    <collision>
+      <origin xyz="0 0 ${z_motor_size/2}" />
+      <geometry>
+        <box size="${x_motor_size} ${y_motor_size} ${z_motor_size}" />
+      </geometry>
+    </collision>
+    <xacro:inertial_box mass="${motor_mass}" x="${x_motor_size}" y="${y_motor_size}"
+      z="${z_motor_size}">
+      <origin xyz="0 0 ${z_motor_size/2}" />
+    </xacro:inertial_box>
+  </link>
   <!-- LEFT WHEEL -->
   <joint name="left_wheel_joint" type="continuous">
-    <parent link="base_link" />
+    <parent link="left_motor" />
     <child link="left_wheel" />
-    <origin xyz="-${2*x_chassis_size /6} ${y_chassis_size/2 + drive_wheel_length/2} 0"
+    <origin xyz="0 ${-y_motor_size} 0"
       rpy="-${pi/2} 0 0" />
     <axis xyz="0 0 1" />
@@ -90,9 +116,35 @@
     <material>Gazebo/Blue</material>
   </gazebo>
+  <!-- RIGHT MOTOR -->
+  <joint name="right_motor_joint" type="continuous">
+    <parent link="base_link" />
+    <child link="right_motor" />
+    <origin xyz="-${2*x_chassis_size /6} ${y_chassis_size/2} 0"
+      rpy="0 0 0" />
+    <axis xyz="0 0 -1" />
+  </joint>
+  <link name="right_motor">
+    <visual>
+      <geometry>
+        <box size="${x_motor_size} ${y_motor_size} ${z_motor_size}" />
+      </geometry>
+      <material name="blue" />
+    </visual>
+    <collision>
+      <origin xyz="0 0 ${z_motor_size/2}" />
+      <geometry>
+        <box size="${x_motor_size} ${y_motor_size} ${z_motor_size}" />
+      </geometry>
+    </collision>
+    <xacro:inertial_box mass="${motor_mass}" x="${x_motor_size}" y="${y_motor_size}"
+      z="${z_motor_size}">
+      <origin xyz="0 0 ${z_motor_size/2}" />
+    </xacro:inertial_box>
+  </link>
   <!-- RIGHT WHEEL -->
   <joint name="right_wheel_joint" type="continuous">
-    <parent link="base_link" />
+    <parent link="right_motor" />
     <child link="right_wheel" />
-    <origin xyz="-${2*x_chassis_size /6} -${y_chassis_size/2 + drive_wheel_length/2} 0"
+    <origin xyz="0 ${y_motor_size} 0"
       rpy="${pi/2} 0 0" />
     <axis xyz="0 0 -1" />

File: description/settings/frame_properties.xacro (robot description, xacro)
@@ -14,4 +14,9 @@
   <xacro:property name="drive_wheel_length" value="0.04" />
   <xacro:property name="drive_wheel_mass" value="2" />
+  <!-- MOTOR -->
+  <xacro:property name="x_motor_size" value="0.05" />
+  <xacro:property name="y_motor_size" value="0.05" />
+  <xacro:property name="z_motor_size" value="0.05" />
+  <xacro:property name="motor_mass" value="1" />
   <!-- CASTER WHEELS-->
   <xacro:property name="caster_wheel_radius" value="0.055" />

Commit message: fix bug

File: description/robot_core.xacro (robot description, xacro)
@@ -63,5 +63,5 @@
   </link>
   <!-- LEFT MOTOR -->
-  <joint name="left_motor_joint" type="continuous">
+  <joint name="left_motor_joint" type="fixed">
     <parent link="base_link" />
     <child link="left_motor" />
@@ -117,5 +117,5 @@
   </gazebo>
   <!-- RIGHT MOTOR -->
-  <joint name="right_motor_joint" type="continuous">
+  <joint name="right_motor_joint" type="fixed">
     <parent link="base_link" />
     <child link="right_motor" />
