Commit message: add basic lidar

File: description/lidar.xacro (robot description, xacro)
@@ -1,3 +1,20 @@
 <?xml version="1.0"?>
 <robot xmlns:xacro="http://www.ros.org/wiki/xacro">
+  <!-- INCLUDE -->
+  <xacro:include filename="settings/materials.xacro" />
+  <xacro:include filename="settings/frame_properties.xacro" />
+  <!-- LASER -->
+  <joint name="laser_joint" type="fixed">
+    <parent link="chassis" />
+    <child link="laser_frame" />
+    <origin xyz="0 0 0" rpy="0 0 0 " />
+  </joint>
+  <link name="laser_frame">
+    <visual>
+      <geometry>
+        <cylinder radius="0.05" length="0.04" />
+      </geometry>
+      <material name="red" />
+    </visual>
+  </link>
 </robot>

File: description/settings/materials.xacro (robot description, xacro)
@@ -14,3 +14,6 @@
     <color rgba="0 0 0 1" />
   </material>
+  <material name="red">
+    <color rgba="1 0 0 1" />
+  </material>
 </robot>

Commit message: add lidar collision

File: description/lidar.xacro (robot description, xacro)
@@ -4,4 +4,5 @@
   <xacro:include filename="settings/materials.xacro" />
   <xacro:include filename="settings/frame_properties.xacro" />
+  <xacro:include filename="inertial_macros.xacro" />
   <!-- LASER -->
   <joint name="laser_joint" type="fixed">
@@ -17,4 +18,12 @@
       <material name="red" />
     </visual>
+    <collision>
+      <geometry>
+        <cylinder radius="0.05" length="0.04" />
+      </geometry>
+    </collision>
+    <xacro:inertial_cylinder mass="0.1" radius="0.05" length="0.04">
+      <origin xyz="0 0 0" rpy="0 0 0" />
+    </xacro:inertial_cylinder>
   </link>
 </robot>

Commit message: move lidar frame properties to settings

File: description/lidar.xacro (robot description, xacro)
@@ -5,10 +5,10 @@
     <parent link="chassis" />
     <child link="laser_frame" />
-    <origin xyz="0 0 0" rpy="0 0 0 " />
+    <origin xyz="0 0 ${z_chassis_size}" rpy="0 0 0 " />
   </joint>
   <link name="laser_frame">
     <visual>
       <geometry>
-        <cylinder radius="0.05" length="0.04" />
+        <cylinder radius="${lidar_frame_radius}" length="${lidar_frame_length}" />
       </geometry>
       <material name="red" />
@@ -16,8 +16,9 @@
     <collision>
       <geometry>
-        <cylinder radius="0.05" length="0.04" />
+        <cylinder radius="${lidar_frame_radius}" length="${lidar_frame_length}" />
       </geometry>
     </collision>
-    <xacro:inertial_cylinder mass="0.1" radius="0.05" length="0.04">
+    <xacro:inertial_cylinder mass="${lidar_mass}" radius="${lidar_frame_radius}"
+      length="${lidar_frame_length}">
       <origin xyz="0 0 0" rpy="0 0 0" />
     </xacro:inertial_cylinder>

File: description/settings/frame_properties.xacro (robot description, xacro)
@@ -14,4 +14,8 @@
   <xacro:property name="caster_wheel_length" value="0.02" />
   <xacro:property name="caster_wheel_mass" value="1" />
+  <!-- LIDAR -->
+  <xacro:property name="lidar_frame_radius" value="0.05" />
+  <xacro:property name="lidar_frame_length" value="0.04" />
+  <xacro:property name="lidar_mass" value="0.1" />
   <!-- SPEED -->
   <xacro:property name="max_wheel_torque" value="100" />

Commit message: add gazebo lidar sim

File: description/lidar.xacro (robot description, xacro)
@@ -5,4 +5,5 @@
     <parent link="chassis" />
     <child link="laser_frame" />
+    <!-- <origin xyz="0 0 ${z_chassis_size}" rpy="0 0 0 " /> -->
     <origin xyz="0 0 ${z_chassis_size}" rpy="0 0 0 " />
   </joint>
@@ -24,3 +25,33 @@
     </xacro:inertial_cylinder>
   </link>
+  <gazebo reference="laser_frame">
+    <material>Gazebo/Red</material>
+    <sensor name="laser" type="ray">
+      <pose>0 0 0 0 0 0</pose>
+      <visualize>true</visualize>
+      <update_rate>10</update_rate>
+      <ray>
+        <scan>
+          <horizontal>
+            <samples>360</samples>
+            <resolution>1</resolution>
+            <min_angle>-3.14</min_angle>
+            <max_angle>3.14</max_angle>
+          </horizontal>
+        </scan>
+        <range>
+          <min>0.3</min>
+          <max>12.0</max>
+          <resolution>0.01</resolution>
+        </range>
+      </ray>
+      <plugin name="laser_controller" filename="libgazebo_ros_ray_sensor.so">
+        <ros>
+          <argument>~/out:=scan</argument>
+        </ros>
+        <output_type>sensor_msgs/LaserScan</output_type>
+        <frame_name>laser_frame</frame_name>
+      </plugin>
+    </sensor>
+  </gazebo>
 </robot>

Commit message: update config

File: description/lidar.xacro (robot description, xacro)
@@ -33,14 +33,14 @@
         <scan>
           <horizontal>
-            <samples>360</samples>
-            <resolution>1</resolution>
-            <min_angle>-3.14</min_angle>
-            <max_angle>3.14</max_angle>
+            <samples>${lidar_samples}</samples>
+            <resolution>${lidar_resolution}</resolution>
+            <min_angle>${lidar_min_angle}</min_angle>
+            <max_angle>${lidar_max_angle}</max_angle>
           </horizontal>
         </scan>
         <range>
-          <min>0.3</min>
-          <max>12.0</max>
-          <resolution>0.01</resolution>
+          <min>${lidar_min_range}</min>
+          <max>${lidar_max_range}</max>
+          <resolution>${lidar_range_resolution}</resolution>
         </range>
       </ray>

File: description/settings/frame_properties.xacro (robot description, xacro)
@@ -18,4 +18,11 @@
   <xacro:property name="lidar_frame_length" value="0.04" />
   <xacro:property name="lidar_mass" value="0.1" />
+  <xacro:property name="lidar_samples" value="360" />
+  <xacro:property name="lidar_resolution" value="1" />
+  <xacro:property name="lidar_min_angle" value="-3.14" />
+  <xacro:property name="lidar_max_angle" value="3.14" />
+  <xacro:property name="lidar_min_range" value="0.3" />
+  <xacro:property name="lidar_max_range" value="12" />
+  <xacro:property name="lidar_range_resolution" value="0.01" />
   <!-- CAMERA -->
   <xacro:property name="x_camera_size" value="0.05" />

Commit message: change lidar position to middle of robot's handle

File: description/lidar.xacro (robot description, xacro)
@@ -1,9 +1,35 @@
 <?xml version="1.0"?>
 <robot xmlns:xacro="http://www.ros.org/wiki/xacro">
+  <!-- LASER BASE -->
+  <joint name="laser_base_joint" type="fixed">
+    <parent link="handle" />
+    <child link="laser_base_frame" />
+    <origin xyz="${x_handle_size} 0 ${13*z_handle_size/20}" rpy="0 0 0 " />
+  </joint>
+  <link name="laser_base_frame">
+    <visual>
+      <geometry>
+        <box size="${x_lidar_base_size} ${y_lidar_base_size} ${z_lidar_base_size}" />
+      </geometry>
+      <material name="red" />
+    </visual>
+    <collision>
+      <geometry>
+        <box size="${x_lidar_base_size} ${y_lidar_base_size} ${z_lidar_base_size}" />
+      </geometry>
+    </collision>
+    <xacro:inertial_box mass="${motor_mass}" x="${x_lidar_base_size}" y="${y_lidar_base_size}"
+      z="${z_lidar_base_size}">
+      <origin xyz="0 0 0" />
+    </xacro:inertial_box>
+  </link>
+  <gazebo reference="laser_base_frame">
+    <material>Gazebo/Blue</material>
+  </gazebo>
   <!-- LASER -->
   <joint name="laser_joint" type="fixed">
-    <parent link="handle" />
+    <parent link="laser_base_frame" />
     <child link="laser_frame" />
-    <origin xyz="0 0 ${z_handle_size + 0.02}" rpy="0 0 0 " />
+    <origin xyz="0 0 ${z_lidar_base_size}" rpy="0 0 0 " />
   </joint>
   <link name="laser_frame">

File: description/settings/frame_properties.xacro (robot description, xacro)
@@ -24,4 +24,7 @@
   <xacro:property name="caster_wheel_mass" value="1" />
   <!-- LIDAR -->
+  <xacro:property name="x_lidar_base_size" value="0.15" />
+  <xacro:property name="y_lidar_base_size" value="0.20" />
+  <xacro:property name="z_lidar_base_size" value="0.05" />
   <xacro:property name="lidar_frame_radius" value="0.05" />
   <xacro:property name="lidar_frame_length" value="0.04" />
