Commit message: increse max spd range

File: description/settings/frame_properties.xacro (robot description, xacro)
@@ -34,5 +34,5 @@
   <xacro:property name="max_wheel_torque" value="100" />
   <xacro:property name="max_acceleration" value="5.0" />
-  <xacro:property name="wheel_max_speed" value="10.0" />
-  <xacro:property name="wheel_min_speed" value="-10.0" />
+  <xacro:property name="wheel_max_speed" value="100.0" />
+  <xacro:property name="wheel_min_speed" value="-100.0" />
 </robot>

Commit message: change wheel min and max speed

File: description/settings/frame_properties.xacro (robot description, xacro)
@@ -34,5 +34,5 @@
   <xacro:property name="max_wheel_torque" value="100" />
   <xacro:property name="max_acceleration" value="5.0" />
-  <xacro:property name="wheel_max_speed" value="100.0" />
-  <xacro:property name="wheel_min_speed" value="-100.0" />
+  <xacro:property name="wheel_max_speed" value="275.0" />
+  <xacro:property name="wheel_min_speed" value="-275.0" />
 </robot>

Commit message: lidar config

File: description/settings/frame_properties.xacro (robot description, xacro)
@@ -28,9 +28,9 @@
   <xacro:property name="lidar_mass" value="0.1" />
   <xacro:property name="lidar_samples" value="360" />
-  <xacro:property name="lidar_resolution" value="1" />
+  <xacro:property name="lidar_resolution" value="0.0174533" />
   <xacro:property name="lidar_min_angle" value="-3.14" />
   <xacro:property name="lidar_max_angle" value="3.14" />
-  <xacro:property name="lidar_min_range" value="0.3" />
-  <xacro:property name="lidar_max_range" value="12" />
+  <xacro:property name="lidar_min_range" value="0.12" />
+  <xacro:property name="lidar_max_range" value="3.5" />
   <xacro:property name="lidar_range_resolution" value="0.01" />
   <!-- CAMERA -->

Commit message: update wheel properties

File: description/settings/frame_properties.xacro (robot description, xacro)
@@ -48,8 +48,8 @@
   <xacro:property name="max_depth" value="100.0" />
   <!-- SPEED -->
-  <xacro:property name="max_wheel_torque" value="100" />
-  <xacro:property name="max_acceleration" value="5.0" />
+  <xacro:property name="max_wheel_torque" value="0.883" />
+  <xacro:property name="max_acceleration" value="1.48" />
   <!-- ROTATION SPEED -->
-  <xacro:property name="wheel_max_speed" value="4.18" />
-  <xacro:property name="wheel_min_speed" value="-4.18" />
+  <xacro:property name="wheel_max_speed" value="1.848" />
+  <xacro:property name="wheel_min_speed" value="-1.848" />
 </robot>

Commit message: change lidar min max angle

File: description/settings/frame_properties.xacro (robot description, xacro)
@@ -32,6 +32,6 @@
   <xacro:property name="lidar_samples" value="360" />
   <xacro:property name="lidar_resolution" value="0.0174533" />
-  <xacro:property name="lidar_min_angle" value="-3.14" />
-  <xacro:property name="lidar_max_angle" value="3.14" />
+  <xacro:property name="lidar_min_angle" value="-1.57" />
+  <xacro:property name="lidar_max_angle" value="1.57" />
   <xacro:property name="lidar_min_range" value="0.12" />
   <xacro:property name="lidar_max_range" value="3.5" />
